File: BusinessCard_Hardware/BusinessCards.kicad_pcb (KiCad board)
At the start: 2 copper layers, 88.9 x 50.8 mm, 16 parts, among them SW1 SW_SPST, U1 L7805

Commit message: Created BOM
Other:
- board text added: "(314) 546-6228 a.vanhorn@mst.edu"
- board text removed: "(314) 546-6228 a.vanhorn@umsystem.edu"
Changed lines of the file:
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@@
       (outputformat 1)
       (mirror false)
-      (drillshape 1)
+      (drillshape 0)
       (scaleselection 1)
-      (outputdirectory ""))
+      (outputdirectory "Gerbs/"))
   )
   (net 0 "")
@@
     (effects (font (size 5.08 5.08) (thickness 0.9525)))
   )
-  (gr_text "(314) 546-6228\na.vanhorn@umsystem.edu" (at 147.32 96.52) (layer F.SilkS)
+  (gr_text "(314) 546-6228\na.vanhorn@mst.edu" (at 147.32 96.52) (layer F.SilkS)
     (effects (font (size 2.54 2.54) (thickness 0.254)))
   )

Commit message: fixed battery holder outline
Parts:
- moved C1 8.61 mm to (164.3, 55.5), turned to 90 degrees
- moved C2 6.33 mm to (168.9, 55.5), turned to 90 degrees
- moved U1 2.79 mm to (166.6, 64.8)
Routing:
- net +5V: track 55.2 -> 56.9 mm
- net Net-(C1-Pad1): track 23.0 -> 24.2 mm
Other:
- board text added: "B.S. Electrical & Computer Engineering '21 Missouri S&T"
- board text removed: "B.S. Electrical & Computer Engineering '21 Chief Technical Officer - Mars Rover Design Team Missouri S&T"

Commit message: updated gerbs
Other:
- board text added: "Updated: 6/2020"
Changed lines of the file:
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@@
   (general
     (thickness 1.6)
-    (drawings 23)
+    (drawings 24)
     (tracks 53)
     (zones 0)
@@
   )
   (setup
-    (last_trace_width 0.762)
+    (last_trace_width 0.25)
     (user_trace_width 0.381)
     (user_trace_width 0.762)
@@
     )
   )
+  (gr_text "Updated: 6/2020" (at 177.8 99.06) (layer B.SilkS)
+    (effects (font (size 1.5 1.5) (thickness 0.3)) (justify mirror))
+  )
   (gr_text Off (at 142.24 58.42) (layer B.SilkS)
